Commit message: Translate all in-code comments and docs to English
Translate comments, launch-argument descriptions and runtime log
messages from French to English across the package. No functional
code changed; material identifiers in the URDF are left as-is.

File: urdf/slam_robot.urdf.xacro (robot description, xacro)
@@ -1,8 +1,8 @@
 <?xml version="1.0"?>
 <!--
-  URDF du robot SLAM Mecanum.
-  Arbre des frames :
-    base_footprint (projection au sol)
-      └── base_link (centre géométrique du châssis)
+  URDF of the Mecanum SLAM robot.
+  Frame tree:
+    base_footprint (ground projection)
+      └── base_link (geometric center of the chassis)
             ├── wheel_front_left_link
             ├── wheel_front_right_link
@@ -10,42 +10,41 @@
             ├── wheel_rear_right_link
             ├── laser_frame   (YDLIDAR X2)
-            └── imu_link      (MPU-6050 sur l'Arduino)
-  Toutes les dimensions sont regroupées dans les propriétés ci-dessous.
-  Les roues sont attachées par des joints FIXES : elles sont purement
-  visuelles (pas besoin de joint_state_publisher). Si un jour tu veux les
-  voir tourner dans RViz, passe les joints en "continuous" et lance
-  joint_state_publisher.
+            └── imu_link      (MPU-6050 on the Arduino)
+  All dimensions are grouped in the properties below.
+  The wheels are attached with FIXED joints: they are purely visual (no
+  joint_state_publisher needed). If you ever want to see them spin in RViz,
+  switch the joints to "continuous" and run joint_state_publisher.
 -->
 <robot xmlns:xacro="http://www.ros.org/wiki/xacro" name="slam_robot">
-  <!-- ================= DIMENSIONS À AJUSTER ================= -->
-  <!-- Demi-empattements : distance du centre du châssis à l'AXE des roues.
-       WHEELBASE_X = distance avant/arrière, WHEELBASE_Y = gauche/droite
-       (centre du châssis -> centre de la roue, PAS roue à roue). -->
-  <xacro:property name="wheelbase_x" value="0.15"/>   <!-- TODO: À MESURER (m) -->
-  <xacro:property name="wheelbase_y" value="0.15"/>   <!-- TODO: À MESURER (m) -->
-  <!-- Roues Mecanum Ø97 mm -->
+  <!-- ================= DIMENSIONS TO ADJUST ================= -->
+  <!-- Half-wheelbases: distance from the chassis center to the wheel AXIS.
+       WHEELBASE_X = front/rear distance, WHEELBASE_Y = left/right
+       (chassis center -> wheel center, NOT wheel to wheel). -->
+  <xacro:property name="wheelbase_x" value="0.15"/>   <!-- TODO: MEASURE (m) -->
+  <xacro:property name="wheelbase_y" value="0.15"/>   <!-- TODO: MEASURE (m) -->
+  <!-- Mecanum wheels, 97 mm diameter -->
   <xacro:property name="wheel_radius" value="0.0485"/>
-  <xacro:property name="wheel_width"  value="0.040"/>  <!-- TODO: À MESURER (m) -->
-  <!-- Châssis (simple boîte pour le visuel) -->
-  <xacro:property name="chassis_length" value="0.28"/> <!-- TODO: À MESURER (m) -->
-  <xacro:property name="chassis_width"  value="0.24"/> <!-- TODO: À MESURER (m) -->
-  <xacro:property name="chassis_height" value="0.10"/> <!-- TODO: À MESURER (m) -->
-  <!-- Hauteur du CENTRE du châssis par rapport au sol -->
-  <xacro:property name="chassis_z_offset" value="${wheel_radius + 0.02}"/> <!-- TODO: À MESURER -->
-  <!-- LiDAR : position du centre optique par rapport à base_link.
-       Le X2 est supposé centré sur le châssis (x=0, y=0). -->
-  <xacro:property name="lidar_x" value="0.0"/>         <!-- TODO: À MESURER si décentré (m) -->
-  <xacro:property name="lidar_y" value="0.0"/>         <!-- TODO: À MESURER si décentré (m) -->
-  <!-- Hauteur du plan laser PAR RAPPORT AU SOL, on retranche l'offset du châssis -->
-  <xacro:property name="lidar_height_from_ground" value="0.20"/> <!-- TODO: À MESURER (m) -->
+  <xacro:property name="wheel_width"  value="0.040"/>  <!-- TODO: MEASURE (m) -->
+  <!-- Chassis (simple box for the visual) -->
+  <xacro:property name="chassis_length" value="0.28"/> <!-- TODO: MEASURE (m) -->
+  <xacro:property name="chassis_width"  value="0.24"/> <!-- TODO: MEASURE (m) -->
+  <xacro:property name="chassis_height" value="0.10"/> <!-- TODO: MEASURE (m) -->
+  <!-- Height of the chassis CENTER above the ground -->
+  <xacro:property name="chassis_z_offset" value="${wheel_radius + 0.02}"/> <!-- TODO: MEASURE -->
+  <!-- LiDAR: position of the optical center relative to base_link.
+       The X2 is assumed centered on the chassis (x=0, y=0). -->
+  <xacro:property name="lidar_x" value="0.0"/>         <!-- TODO: MEASURE if off-center (m) -->
+  <xacro:property name="lidar_y" value="0.0"/>         <!-- TODO: MEASURE if off-center (m) -->
+  <!-- Laser plane height RELATIVE TO THE GROUND; subtract the chassis offset -->
+  <xacro:property name="lidar_height_from_ground" value="0.20"/> <!-- TODO: MEASURE (m) -->
   <xacro:property name="lidar_z" value="${lidar_height_from_ground - chassis_z_offset}"/>
-  <!-- Rotation du LiDAR autour de Z si son "avant" n'est pas aligné avec
-       l'avant du robot (ex : 3.14159 s'il est monté à l'envers). -->
-  <xacro:property name="lidar_yaw" value="0.0"/>       <!-- TODO: À VÉRIFIER (rad) -->
-  <!-- IMU MPU-6050 : position par rapport à base_link -->
-  <xacro:property name="imu_x" value="0.0"/>           <!-- TODO: À MESURER (m) -->
-  <xacro:property name="imu_y" value="0.0"/>           <!-- TODO: À MESURER (m) -->
-  <xacro:property name="imu_z" value="0.0"/>           <!-- TODO: À MESURER (m) -->
-  <!-- ================= COULEURS ================= -->
+  <!-- LiDAR rotation about Z if its "front" is not aligned with the robot's
+       front (e.g. 3.14159 if it is mounted backwards). -->
+  <xacro:property name="lidar_yaw" value="0.0"/>       <!-- TODO: CHECK (rad) -->
+  <!-- IMU MPU-6050: position relative to base_link -->
+  <xacro:property name="imu_x" value="0.0"/>           <!-- TODO: MEASURE (m) -->
+  <xacro:property name="imu_y" value="0.0"/>           <!-- TODO: MEASURE (m) -->
+  <xacro:property name="imu_z" value="0.0"/>           <!-- TODO: MEASURE (m) -->
+  <!-- ================= COLORS ================= -->
   <material name="gris_chassis"><color rgba="0.4 0.4 0.4 1.0"/></material>
   <material name="noir_roue"><color rgba="0.1 0.1 0.1 1.0"/></material>
@@ -53,6 +52,6 @@
   <material name="rouge_imu"><color rgba="0.8 0.1 0.1 1.0"/></material>
   <!-- ================= BASE ================= -->
-  <!-- base_footprint : projection de base_link au sol (z = 0).
-       C'est la frame de référence utilisée par slam_toolbox et Nav2. -->
+  <!-- base_footprint: projection of base_link onto the ground (z = 0).
+       This is the reference frame used by slam_toolbox and Nav2. -->
   <link name="base_footprint"/>
   <joint name="base_footprint_to_base_link" type="fixed">
@@ -69,7 +68,7 @@
     </visual>
   </link>
-  <!-- ================= ROUES ================= -->
-  <!-- Macro roue : cylindre orienté axe Y (rotation de 90° autour de X).
-       reflect_x = +1 avant / -1 arrière ; reflect_y = +1 gauche / -1 droite -->
+  <!-- ================= WHEELS ================= -->
+  <!-- Wheel macro: cylinder oriented along the Y axis (90 deg rotation about X).
+       reflect_x = +1 front / -1 rear ; reflect_y = +1 left / -1 right -->
   <xacro:macro name="roue" params="prefix reflect_x reflect_y">
     <link name="wheel_${prefix}_link">
@@ -85,5 +84,5 @@
       <parent link="base_link"/>
       <child link="wheel_${prefix}_link"/>
-      <!-- La roue est au niveau de son axe : z ramené à la hauteur de l'axe -->
+      <!-- The wheel sits at its axis level: z brought to the axis height -->
       <origin xyz="${reflect_x * wheelbase_x} ${reflect_y * wheelbase_y} ${wheel_radius - chassis_z_offset}"
               rpy="0 0 0"/>
@@ -98,5 +97,5 @@
     <visual>
       <geometry>
-        <!-- Approximation du boîtier du YDLIDAR X2 -->
+        <!-- Approximation of the YDLIDAR X2 housing -->
         <cylinder radius="0.035" length="0.04"/>
       </geometry>
